Commit message: camera lidar calibration

File: src/wheelchair_description/urdf/wheelchair_rs.xacro (robot description, xacro)
@@ -4,4 +4,5 @@
   <xacro:include filename="$(find wheelchair_description)/urdf/links_joints.xacro" />
   <xacro:include filename="$(find wheelchair_description)/urdf/wheelchair_gazebo.xacro" />
+	<!-- <xacro:include filename="$(find azure_kinect_ros_driver)/urdf/azure_kinect.urdf.xacro" /> -->
   <xacro:include filename="$(find wheelchair_description)/urdf/_d435.xacro" />
   <xacro:arg name="use_nominal_extrinsics" default="false"/>
@@ -12,5 +13,5 @@
       <parent link="base_link"/>
       <child link="chassis" />
-      <origin xyz="0 0 0.2" rpy="0 0 0"/>
+      <origin xyz="0.22 0.0 0.2" rpy="0 0 0"/>
     </joint>
     <link name='chassis'>
@@ -170,32 +171,14 @@
                    material="black"
                    filename="package://wheelchair_description/meshes/rplidar.dae" scale="1 1 1"/>
-<!-- joint between chassis and lidar -->
-      <xacro:f_joint name="chassis_to_rplidar"
+    <!-- new config -->
+      <xacro:f_joint name="base_link_to_rplidar"
                type="fixed"
                axis_xyz="0 0 0"
-               origin_rpy="0 0 -1.57" origin_xyz="0.23 0 -0.15"
-               parent="chassis" child="rplidar" />
+               origin_rpy="0 0 0" origin_xyz="0.80 0 0"
+               parent="base_link" child="rplidar" />
 <!--Real_Sense-->
-    <!--D435 with tilted angle as in real wheelchair-->
-      <!--xacro:sensor_d435 parent="base_link">
-        <origin xyz="-0.23 0 0.860" rpy="0 -0.24 0"/>
-      </xacro:sensor_d435-->
-<!--Labtest 3, decent alignment-->
-     <!--xacro:sensor_d455 parent="base_link" name="camera2">
-        <origin xyz="-0.23 0 0.860" rpy="0 0 0"/>
-      </xacro:sensor_d455>
-      <xacro:sensor_d455 parent="camera_base_rod" name="camera1">
-        <origin xyz="0.53 -0.25 -0.58" rpy="-0.005 -0.11 -0.03"/>
-      </xacro:sensor_d455-->
       <xacro:sensor_d435 parent="base_link" name="camera">
-        <origin xyz="0.20 -0.24 0.50" rpy="0 -0.01 0"/>
+        <origin xyz="0.05 0 1.31" rpy="0 0.261799 -0.03"/>
       </xacro:sensor_d435>
-      <!--xacro:sensor_d455 parent="camera_base_rod" name="camera1">
-        <origin xyz="0.60 -0.34 -0.50" rpy="0 -0.01 0"/>
-      </xacro:sensor_d455-->
-      <!--xacro:sensor_d455 parent="camera2_link" name="camera1">
-        <origin xyz="0.60 -0.34 -0.50" rpy="0 -0.01 0"/>
-      </xacro:sensor_d455-->
-    <!--Gazebo Plugin-->
     <gazebo>
       <plugin name="gazebo_ros_control" filename="libgazebo_ros_control.so">

File: src/wheelchair_description/urdf/wheelchair_zed.xacro (robot description, xacro)
@@ -171,10 +171,4 @@
                    material="black"
                    filename="package://wheelchair_description/meshes/rplidar.dae" scale="1 1 1"/>
-<!-- joint between chassis and lidar -->
-      <!-- <xacro:f_joint name="chassis_to_rplidar"
-               type="fixed"
-               axis_xyz="0 0 0"
-               origin_rpy="0 0 -1.57" origin_xyz="0.23 0 -0.15"
-               parent="chassis" child="rplidar" /> -->
     <!-- new config -->
       <xacro:f_joint name="base_link_to_rplidar"
@@ -186,19 +180,4 @@
       rpy="0 -0.25 0") -->
 <!--Real_Sense-->
-    <!--D435 with tilted angle as in real wheelchair-->
-      <!--xacro:sensor_d435 parent="base_link">
-        <origin xyz="-0.23 0 0.860" rpy="0 -0.24 0"/>
-      </xacro:sensor_d435-->
-<!--Labtest 3, decent alignment-->
-     <!--xacro:sensor_d455 parent="base_link" name="camera2">
-        <origin xyz="-0.23 0 0.860" rpy="0 0 0"/>
-      </xacro:sensor_d455>
-      <xacro:sensor_d455 parent="camera_base_rod" name="camera1">
-        <origin xyz="0.53 -0.25 -0.58" rpy="-0.005 -0.11 -0.03"/>
-      </xacro:sensor_d455-->
-      <!--use this if not using azure-->
-      <!-- <xacro:sensor_d435 parent="base_link" name="camera">
-        <origin xyz="-0.08 -0.1 1.30" rpy="0 0.14 0.067"/>
-      </xacro:sensor_d435> -->
   <xacro:include filename="$(find zed_wrapper)/urdf/zed_macro.urdf.xacro" />
   <xacro:zed_camera name="zed2i" parent="base_link">
@@ -207,16 +186,4 @@
       rpy="0 0.22 0"/>
   </xacro:zed_camera>
-    <!-- <joint name="base_link_to_camera" type="fixed">
-	    <axis xyz="0 0 0" />
-      <origin xyz="0.53 -0.24 0.30" rpy="0 0.035 0.040"/>
-      <parent link="base_link" />
-     <child link="camera_base" />
-    </joint> -->
-      <!--xacro:sensor_d455 parent="camera_base_rod" name="camera1">
-        <origin xyz="0.60 -0.34 -0.50" rpy="0 -0.01 0"/>
-      </xacro:sensor_d455-->
-      <!--xacro:sensor_d455 parent="camera2_link" name="camera1">
-        <origin xyz="0.60 -0.34 -0.50" rpy="0 -0.01 0"/>
-      </xacro:sensor_d455-->
     <!--Gazebo Plugin-->
     <gazebo>
